File: hardware/haptics-circuit/haptics.kicad_sch (KiCad schematic)
At the start: 9 parts, among them M1 Motor_DC, U1 NJU7044D, U2 TB6612FNG Breakout, U3 ESP32-DevKitC

Commit message: Schematic: student version without reconstruction notes
The circuit was confirmed correct, so the drawing, its README and the
circuit page no longer carry the notes about how it was reconstructed
and what was assumed. The JTAG pin note and the unused op-amp note stay.

Co-Authored-By: Claude Opus 5.5 (1M context) <noreply@anthropic.com>
Other:
- note added: "補足 ・JTAG デバッガ(FT232H、緑の基板)の配線は省略。ESP32 の IO12=TDI、IO13=TCK、IO14=TMS、IO15=TDO と GND につながる。 ・U1 の A・B・C 回路は使わない。"
- note removed: "起こし方と確認事項 ・2026年度に、完成品の写真とファームウェア(ICTEx5ActiveHaptic の main.c)から起こした。元の回路図は残っていない。 ・R4(FSR)の、U1 につながらない側の端子は、写真では電源レールのどちらの列か確定できなかった。 ファームウェアが「押すと ADC 値が上がる」前提であることから GND とした(+3V3 だと逆になる)。 ・JTAG デバッガ(FT232H、緑の基板)の配線は省略。ESP32 の IO12=TDI、IO13=TCK、IO14=TMS、IO15=TDO と GND につながる。 ・U1 の A・B・C 回路は実物でも未接続(本来は入力を GND か出力につなぐのが望ましい)。"
Changed lines of the file:
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@@
 (kicad_sch (version 20231120) (generator "eeschema") (generator_version "8.0")
 (paper "A4")
-(title_block (title "触覚提示実験 回路図(ActiveHaptic / SoftHaptics)") (date "2026-10-06") (rev "1") (company "情報通信実験第5") (comment 1 "写真とファームウェアから起こした回路。確認事項は図中の注記を参照"))
+(title_block (title "触覚提示実験 回路図(ActiveHaptic / SoftHaptics)") (date "2026-10-06") (rev "1") (company "情報通信実験第5"))
 (symbol (lib_id "ICTEx5:ESP32-DevKitC") (at 60.96 101.60 0) (unit 1) (exclude_from_sim no) (in_bom yes) (on_board yes) (dnp no)
 (property "Reference" "U3" (at 60.96 72.39 0) (effects (font (size 1.27 1.27))))
@@
 (text "センサアンプ(U1 の D 回路)\nVREF = 3.3 V × R2/(R1+R2) = 1.65 V\nADC_OUT = VREF × (1 + RV1/R4)\n押していない(R4 = FSR ≒ ∞)とき ADC_OUT ≒ 1.65 V(ADC 値 1600〜2000)。\n押すと FSR の抵抗が下がって ADC_OUT が上がる。\nRV1 で感度を調整(押したとき約 2500)。RV1 は可変抵抗として使用。" (exclude_from_sim no) (at 101.60 88.90 0) (effects (font (size 1.27 1.27)) (justify left top)))
 (text "モータ駆動(U2)\nIO5 → AIN1、IO17 → AIN2 に 50 kHz の PWM(bdc_motor)。\nIO16 → PWMA は常に High。STBY・VM・VCC は 3.3 V。\nモータと直列の 4.7 Ω(R3)で電流を制限する。" (exclude_from_sim no) (at 101.60 114.30 0) (effects (font (size 1.27 1.27)) (justify left top)))
-(text "起こし方と確認事項\n・2026年度に、完成品の写真とファームウェア(ICTEx5ActiveHaptic の main.c)から起こした。元の回路図は残っていない。\n・R4(FSR)の、U1 につながらない側の端子は、写真では電源レールのどちらの列か確定できなかった。\n  ファームウェアが「押すと ADC 値が上がる」前提であることから GND とした(+3V3 だと逆になる)。\n・JTAG デバッガ(FT232H、緑の基板)の配線は省略。ESP32 の IO12=TDI、IO13=TCK、IO14=TMS、IO15=TDO と GND につながる。\n・U1 の A・B・C 回路は実物でも未接続(本来は入力を GND か出力につなぐのが望ましい)。" (exclude_from_sim no) (at 20.32 167.64 0) (effects (font (size 1.27 1.27)) (justify left top)))
+(text "補足\n・JTAG デバッガ(FT232H、緑の基板)の配線は省略。ESP32 の IO12=TDI、IO13=TCK、IO14=TMS、IO15=TDO と GND につながる。\n・U1 の A・B・C 回路は使わない。" (exclude_from_sim no) (at 20.32 167.64 0) (effects (font (size 1.27 1.27)) (justify left top)))
 (sheet_instances (path "/" (page "1")))
 )
